File: 0026_Soil_Moisture_Module_TLC555.kicad_sch (KiCad schematic)
At the start: 15 parts, among them U1 TLC555xD, U2 XC6206P302

Commit message: Add files via upload
Parts:
- added D2: LED, LED_SMD:LED_0603_1608Metric, symbol Device:LED
- added J2, J3: Screw_Terminal_01x03, TerminalBlock_4Ucon:TerminalBlock_4Ucon_1x03_P3.50mm_Horizontal, symbol Connector:Screw_Terminal_01x03
- added R5: R, Resistor_SMD:R_0603_1608Metric, symbol Device:R
- added U3: ~, Moduler_:pin_header, symbol moduler_pin:air
- C1, C2, C3, C4, C5, C6, C7, C8: footprint (none) -> Capacitor_SMD:C_0603_1608Metric
- D1: footprint Diode_THT:D_DO-35_SOD27_P7.62mm_Horizontal -> Diode_SMD:D_0805_2012Metric
- R1, R2, R3, R4: footprint (none) -> Resistor_SMD:R_0603_1608Metric
Connections:
- net GND: now also D2.1 (K), J2.1 (Pin_1), J2.3 (Pin_3), J3.1 (Pin_1), J3.3 (Pin_3), U3.9
- net SENSOR+: now also J2.2 (Pin_2), J3.2 (Pin_2)
- net SIG: now also U3.12
- net VCC: no longer C5.1, C7.1, U2.3 (VI)
- new net: D2.2 (A), R5.2
- new net +3V3: C5.1, C7.1, R5.1, U2.3 (VI), U3.8
- no-connect marks 0 -> 15
Other:
- note added: "AIR PIN"
- note added: "BUCK"
- note added: "SENSOR"
- moved on the sheet: C1, C2, C3, C4, C5, C6, C7, C8, D1, R1, R2, R3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
